File: hardware/esp_power_with_op.kicad_pcb (KiCad board)
At the start: 2 copper layers, 23 parts, among them J1 CONN_01X04, P1 CONN_01X06, U1 1206NETWORK, U2 MIC920YC5, U3 AP1117

Commit message: add updated files
Routing:
- net GND: track 101.8 -> 92.8 mm
- net (no net): track 0.00 -> 6.50 mm
Other:
- board text added: "esp_power_with_op"
Changed lines of the file:
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@@
     (area 27.872 23.230999 99.355 51.266)
     (thickness 1.6)
-    (drawings 12)
-    (tracks 170)
+    (drawings 13)
+    (tracks 176)
     (zones 0)
     (modules 23)
@@
     )
   )
+  (gr_text esp_power_with_op (at 36.195 33.02) (layer F.Cu)
+    (effects (font (size 0.762 0.762) (thickness 0.1905)))
+  )
   (gr_text 1ux4 (at 53.11 37.83) (layer F.Cu)
     (effects (font (size 0.8128 0.8128) (thickness 0.2032)))
@@
     (effects (font (size 0.8128 0.8128) (thickness 0.2032)))
   )
+  (segment (start 32.385 49.53) (end 32.385 48.895) (width 0.3302) (layer F.Cu) (net 0))
+  (segment (start 33.02 49.53) (end 32.385 49.53) (width 0.3302) (layer F.Cu) (net 0))
+  (segment (start 33.655 48.895) (end 33.02 49.53) (width 0.3302) (layer F.Cu) (net 0))
+  (segment (start 33.655 48.26) (end 33.655 48.895) (width 0.3302) (layer F.Cu) (net 0))
+  (segment (start 33.02 48.26) (end 33.655 48.26) (width 0.3302) (layer F.Cu) (net 0))
+  (segment (start 32.385 48.895) (end 33.02 48.26) (width 0.3302) (layer F.Cu) (net 0))
+  (segment (start 33.655 48.26) (end 33.655 47.625) (width 0.3302) (layer F.Cu) (net 0))
+  (segment (start 33.655 47.625) (end 34.29 48.26) (width 0.3302) (layer F.Cu) (net 0))
+  (segment (start 34.29 48.26) (end 33.655 48.26) (width 0.3302) (layer F.Cu) (net 0))
   (segment (start 42.902 41.783) (end 42.521 41.783) (width 0.3302) (layer F.Cu) (net 1))
   (segment (start 43.561 44.212) (end 42.902 43.553) (width 0.3302) (layer F.Cu) (net 1))
@@
   (segment (start 42.95 50.419) (end 41.021 48.49) (width 0.3556) (layer F.Cu) (net 8))
   (segment (start 76.962 47.117) (end 73.66 50.419) (width 0.3556) (layer F.Cu) (net 8))
-  (segment (start 33.401 45.212) (end 35.56 45.212) (width 0.3556) (layer F.Cu) (net 8))
-  (segment (start 35.56 45.212) (end 38.838 48.49) (width 0.3556) (layer F.Cu) (net 8))
-  (segment (start 38.838 48.49) (end 41.021 48.49) (width 0.3556) (layer F.Cu) (net 8))
   (segment (start 79.116 46.466) (end 84.382894 46.466) (width 0.3556) (layer F.Cu) (net 8))
   (segment (start 86.782 44.066894) (end 86.782 42.24056) (width 0.3556) (layer F.Cu) (net 8))
