File: hardware/esp_power_with_op.sch (KiCad schematic (older format))
At the start: 23 parts, among them J1 CONN_01X04, P1 CONN_01X06, U1 1206NETWORK, U2 MIC920YC5, U3 AP1117

Commit message: update lighthouse designs
Other:
- note added: "Or compatible with TC75S57FU(TE85L,F)"
Changed lines of the file:
@@
 LIBS:max3010x
 LIBS:l6474
+LIBS:diodearray_sot23-3
+LIBS:mic920yc5
 LIBS:esp_power_with_op-cache
 EELAYER 25 0
@@
 	-1   0    0    1
 $EndComp
+Text Notes 4100 6050 0    60   ~ 0
+Or compatible with TC75S57FU(TE85L,F)
 $EndSCHEMATC
