File: transimpedance2/transimpedance2.kicad_pcb (KiCad board)
At the start: 2 copper layers, 16 parts, among them P1 CONN_01X04, P2 CONN_01X04, P3 10k, U1 DUALOPAMP

Commit message: update the transimpedance esign.
Other:
- board outline added: 28.7 x 15.5 mm
Changed lines of the file:
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@@
-(kicad_pcb (version 4) (host pcbnew 4.0.2+dfsg1-stable)
+(kicad_pcb (version 4) (host pcbnew 4.0.6-e0-6349~53~ubuntu16.04.1)
   (general
     (links 34)
     (no_connects 0)
-    (area 35.839799 30.9245 67.487401 46.233442)
+    (area 35.839799 31.1023 67.487401 47.192001)
     (thickness 1.6)
-    (drawings 15)
+    (drawings 31)
     (tracks 106)
     (zones 0)
@@
     (visible_elements FFFFFF7F)
     (pcbplotparams
-      (layerselection 0x00000_00000001)
+      (layerselection 0x010f8_80000001)
       (usegerberextensions false)
       (excludeedgelayer false)
@@
       (padsonsilk false)
       (subtractmaskfromsilk false)
-      (outputformat 2)
+      (outputformat 1)
       (mirror false)
       (drillshape 0)
       (scaleselection 1)
-      (outputdirectory ""))
+      (outputdirectory transimpedance2))
   )
   (net 0 "")
@@
       (net 4 GND))
   )
+  (gr_text esp8266lighthouse (at 43.03 46.225) (layer F.SilkS)
+    (effects (font (size 0.762 0.762) (thickness 0.1905)))
+  )
+  (gr_text transimpedance2 (at 60.83 46.225) (layer F.SilkS)
+    (effects (font (size 0.762 0.762) (thickness 0.1905)))
+  )
+  (gr_line (start 49.784 46.355) (end 49.276 46.355) (angle 90) (layer F.SilkS) (width 0.2))
+  (gr_line (start 50.292 45.847) (end 49.784 46.355) (angle 90) (layer F.SilkS) (width 0.2))
+  (gr_line (start 50.292 45.339) (end 50.292 45.847) (angle 90) (layer F.SilkS) (width 0.2))
+  (gr_line (start 50.8 45.339) (end 50.292 45.339) (angle 90) (layer F.SilkS) (width 0.2))
+  (gr_line (start 50.292 44.831) (end 50.8 45.339) (angle 90) (layer F.SilkS) (width 0.2))
+  (gr_line (start 50.292 45.339) (end 50.292 44.831) (angle 90) (layer F.SilkS) (width 0.2))
+  (gr_line (start 49.784 45.339) (end 50.292 45.339) (angle 90) (layer F.SilkS) (width 0.2))
+  (gr_line (start 49.276 45.847) (end 49.784 45.339) (angle 90) (layer F.SilkS) (width 0.2))
+  (gr_line (start 49.276 46.355) (end 49.276 45.847) (angle 90) (layer F.SilkS) (width 0.2))
+  (gr_line (start 37.338 31.623) (end 37.592 31.623) (angle 90) (layer Edge.Cuts) (width 0.15))
+  (gr_line (start 37.338 47.117) (end 37.338 31.623) (angle 90) (layer Edge.Cuts) (width 0.15))
+  (gr_line (start 66.04 47.117) (end 37.338 47.117) (angle 90) (layer Edge.Cuts) (width 0.15))
+  (gr_line (start 66.04 31.623) (end 66.04 47.117) (angle 90) (layer Edge.Cuts) (width 0.15))
+  (gr_line (start 37.592 31.623) (end 66.04 31.623) (angle 90) (layer Edge.Cuts) (width 0.15))
   (gr_text 9kvr (at 57.785 41.529) (layer F.Cu)
     (effects (font (size 0.762 0.762) (thickness 0.1905)))
