File: transimpedance3/transimpedance3.sch (KiCad schematic (older format))
At the start: 13 parts, among them P1 CONN_01X04, P2 CONN_01X04, P3 10k, U1 TSV992

Commit message: update tia3
Other:
- note added: "PART / NOISE / FAR / Cost\nPD70-01C/TR7: .159 / .418 / .47\nPD438C: .237 / .550 / .39\nQSD2030F: .216 / .5363 / .30\nBPW34/S-Z: .283 / .6345 /.497\nPD15-216/TR8: UNUSABLE\nVBPW34FAS: .175 / .815 / .778\nVBPW34FASR: .2631 / .644 / .778\nBPW34: .237 / .577 / .62\nPD15-22C/TR8: Unworkable.\nPD15-22B/TR8: Unworkable.\nPD70-TR10: .2063 / .4024 / .41\nBPW46: .247 / .968 / .61\n\nWinners: BPW46, BPW34/S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"
- note removed: "PART / NOISE / FAR / Cost\nPD70-01C/TR7: .159 / .418 / .47\nPD438C: .237 / .550 / .39\nQSD2030F: .216 / .5363 / .30\nBPW34/S-Z: .283 / .6345 /.497\nPD15-216/TR8: UNUSABLE\nBPW34FAS: .175 / .815 / Obsolete?\nVBPW34FASR: .2631 / .644 / .778\nBPW34: .237 / .577 / .62\nPD15-22C/TR8: Unworkable.\nPD15-22B/TR8: Unworkable.\nPD70-TR10: .2063 / .4024 / .41\nBPW46: .247 / .968 / .61\n\nWinners: BPW46, BPW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"
- moved on the sheet: C2, C3
Changed lines of the file:
@@
 L C C2
 U 1 1 58DD4042
-P 8350 1400
-F 0 "C2" H 8375 1500 50  0000 L CNN
-F 1 "10u" H 8375 1300 50  0000 L CNN
-F 2 "C_0805" H 8100 1400 50  0000 C CNN
-F 3 "" H 8350 1400 50  0000 C CNN
-	1    8350 1400
+P 2400 1150
+F 0 "C2" H 2425 1250 50  0000 L CNN
+F 1 "10u" H 2425 1050 50  0000 L CNN
+F 2 "C_0805" H 2150 1150 50  0000 C CNN
+F 3 "" H 2400 1150 50  0000 C CNN
+	1    2400 1150
 	1    0    0    -1
 $EndComp
@@
 L C C3
 U 1 1 58DD40AE
-P 8600 1400
-F 0 "C3" H 8625 1500 50  0000 L CNN
-F 1 "10n" H 8625 1300 50  0000 L CNN
-F 2 "C_0805" H 8638 1250 50  0000 C CNN
-F 3 "" H 8600 1400 50  0000 C CNN
-	1    8600 1400
+P 2650 1150
+F 0 "C3" H 2675 1250 50  0000 L CNN
+F 1 "10n" H 2675 1050 50  0000 L CNN
+F 2 "C_0805" H 2688 1000 50  0000 C CNN
+F 3 "" H 2650 1150 50  0000 C CNN
+	1    2650 1150
 	1    0    0    -1
 $EndComp
@@
 L GND #PWR05
 U 1 1 58DD4181
-P 8350 1550
-F 0 "#PWR05" H 8350 1300 50  0001 C CNN
-F 1 "GND" H 8350 1400 50  0000 C CNN
-F 2 "" H 8350 1550 50  0000 C CNN
-F 3 "" H 8350 1550 50  0000 C CNN
-	1    8350 1550
+P 2400 1300
+F 0 "#PWR05" H 2400 1050 50  0001 C CNN
+F 1 "GND" H 2400 1150 50  0000 C CNN
+F 2 "" H 2400 1300 50  0000 C CNN
+F 3 "" H 2400 1300 50  0000 C CNN
+	1    2400 1300
 	1    0    0    -1
 $EndComp
@@
 L GND #PWR06
 U 1 1 58DD41A1
-P 8600 1550
-F 0 "#PWR06" H 8600 1300 50  0001 C CNN
-F 1 "GND" H 8600 1400 50  0000 C CNN
-F 2 "" H 8600 1550 50  0000 C CNN
-F 3 "" H 8600 1550 50  0000 C CNN
-	1    8600 1550
+P 2650 1300
+F 0 "#PWR06" H 2650 1050 50  0001 C CNN
+F 1 "GND" H 2650 1150 50  0000 C CNN
+F 2 "" H 2650 1300 50  0000 C CNN
+F 3 "" H 2650 1300 50  0000 C CNN
+	1    2650 1300
 	1    0    0    -1
 $EndComp
@@
 L +3.3V #PWR07
 U 1 1 58DD41C1
-P 8350 1250
-F 0 "#PWR07" H 8350 1100 50  0001 C CNN
-F 1 "+3.3V" H 8350 1390 50  0000 C CNN
-F 2 "" H 8350 1250 50  0000 C CNN
-F 3 "" H 8350 1250 50  0000 C CNN
-	1    8350 1250
+P 2400 1000
+F 0 "#PWR07" H 2400 850 50  0001 C CNN
+F 1 "+3.3V" H 2400 1140 50  0000 C CNN
+F 2 "" H 2400 1000 50  0000 C CNN
+F 3 "" H 2400 1000 50  0000 C CNN
+	1    2400 1000
 	1    0    0    -1
 $EndComp
@@
 L +3.3V #PWR08
 U 1 1 58DD41E1
-P 8600 1250
-F 0 "#PWR08" H 8600 1100 50  0001 C CNN
-F 1 "+3.3V" H 8600 1390 50  0000 C CNN
-F 2 "" H 8600 1250 50  0000 C CNN
-F 3 "" H 8600 1250 50  0000 C CNN
-	1    8600 1250
+P 2650 1000
+F 0 "#PWR08" H 2650 850 50  0001 C CNN
+F 1 "+3.3V" H 2650 1140 50  0000 C CNN
+F 2 "" H 2650 1000 50  0000 C CNN
+F 3 "" H 2650 1000 50  0000 C CNN
+	1    2650 1000
 	1    0    0    -1
 $EndComp
@@
 NOTES:\nTESTS Performed with no C1, TSV992\nMaking R4 220k instead of 47k seeems to have little effect, but does make it worse.\nSwitching R1 for 47k just makes it appear drunk. There's some weird feedback thing going on.\n    Like it tuned wrong or something.   Making it 10k quiets the signal a lot.\nREMOVING C4 no apparent impact.\n\nR5=10k, C5=10p -> R5=4.7k, C5=18p =>> Improvement.\nAdding C1=1pF decreases amplitude a little bit but also cleans up edges.\nRemoving C6 seems to reduce amplitude slightly.\n\nFar peak:\nC1 none C6 none => .1238V noise, .998V Far Light\nC1 none C6 1pF    => .1238V noise, .498V Far Light\nC1 1pF  C6 none => .1135V noise, .358V Far Light\nC1 1pF C6 1pF     => .087V Noise, .202V Far Light\n\nRecommendation: Remove C6, C1.\n\nOut of the following op amps...\nTSH82, TSV992, AD8052, TSH22, TSH462,\nTSV992 demolished.
 Text Notes 6900 5650 0    60   ~ 0
-PART / NOISE / FAR / Cost\nPD70-01C/TR7:  .159 / .418 / .47\nPD438C: .237 / .550 / .39\nQSD2030F: .216 / .5363 / .30\nBPW34/S-Z: .283 / .6345 /.497\nPD15-216/TR8: UNUSABLE\nBPW34FAS: .175 / .815 / Obsolete?\nVBPW34FASR: .2631 / .644 / .778\nBPW34: .237 / .577 / .62\nPD15-22C/TR8: Unworkable.\nPD15-22B/TR8: Unworkable.\nPD70-TR10: .2063 / .4024 / .41\nBPW46: .247 / .968 / .61\n\nWinners: BPW46, BPW34/S-Z, BPW34FAS + VBPW34FASR\nMajor Winners: BPW46/VBPW34FAS
+PART / NOISE / FAR / Cost\nPD70-01C/TR7:  .159 / .418 / .47\nPD438C: .237 / .550 / .39\nQSD2030F: .216 / .5363 / .30\nBPW34/S-Z: .283 / .6345 /.497\nPD15-216/TR8: UNUSABLE\nVBPW34FAS: .175 / .815 / .778\nVBPW34FASR: .2631 / .644 / .778\nBPW34: .237 / .577 / .62\nPD15-22C/TR8: Unworkable.\nPD15-22B/TR8: Unworkable.\nPD70-TR10: .2063 / .4024 / .41\nBPW46: .247 / .968 / .61\n\nWinners: BPW46, BPW34/S-Z, BPW34FAS + VBPW34FASR\nMajor Winners: BPW46/VBPW34FAS
 Text Notes 2000 2050 0    60   ~ 0
 BPW46 or VBPW34FAS

Commit message: Update all designs with newest to fab.
Parts:
- removed P1: CONN_01X04, TerminalBlock_Pheonix_MPT-2.54mm_4pol, symbol CONN_01X04
- added J1: PHOTO, Pin_Header_Straight_1x02_Pitch2.54mm, symbol CONN_01X02
- C1: renamed from C5; value 18pF -> 36pF; footprint C_0805 -> C_0603
- C2, C3, R1, R2, R4, R5: footprint C_0805 -> C_0603
- C4: renamed from C7; footprint C_0805 -> C_0603
- P2: value CONN_01X04 -> SYS
Changed lines of the file:
@@
 F 0 "R1" V 3480 2150 50  0000 C CNN
 F 1 "22k" V 3400 2150 50  0000 C CNN
-F 2 "C_0805" H 3400 2550 50  0000 C CNN
+F 2 "C_0603" H 3400 2550 50  0000 C CNN
 F 3 "" H 3400 2150 50  0000 C CNN
 	1    3400 2150
@@
 $EndComp
 $Comp
-L GND #PWR01
+L GND #PWR7
 U 1 1 58DD3F49
 P 4250 2350
-F 0 "#PWR01" H 4250 2100 50  0001 C CNN
+F 0 "#PWR7" H 4250 2100 50  0001 C CNN
 F 1 "GND" H 4250 2200 50  0000 C CNN
 F 2 "" H 4250 2350 50  0000 C CNN
@@
 F 0 "R2" V 4480 1700 50  0000 C CNN
 F 1 "10k" V 4400 1700 50  0000 C CNN
-F 2 "C_0805" V 4330 1700 50  0001 C CNN
+F 2 "C_0603" V 4330 1700 50  0001 C CNN
 F 3 "" H 4400 1700 50  0000 C CNN
 	1    4400 1700
@@
 $EndComp
 $Comp
-L +3.3V #PWR03
+L +3.3V #PWR8
 U 1 1 58DD3FEE
 P 4550 1700
-F 0 "#PWR03" H 4550 1550 50  0001 C CNN
+F 0 "#PWR8" H 4550 1550 50  0001 C CNN
 F 1 "+3.3V" H 4550 1840 50  0000 C CNN
 F 2 "" H 4550 1700 50  0000 C CNN
@@
 $EndComp
 $Comp
-L +3.3V #PWR04
+L +3.3V #PWR9
 U 1 1 58DD4014
 P 5150 2050
-F 0 "#PWR04" H 5150 1900 50  0001 C CNN
+F 0 "#PWR9" H 5150 1900 50  0001 C CNN
 F 1 "+3.3V" H 5150 2190 50  0000 C CNN
 F 2 "" H 5150 2050 50  0000 C CNN
@@
 F 0 "C2" H 2425 1250 50  0000 L CNN
 F 1 "10u" H 2425 1050 50  0000 L CNN
-F 2 "C_0805" H 2150 1150 50  0000 C CNN
+F 2 "C_0603" H 2150 1150 50  0000 C CNN
 F 3 "" H 2400 1150 50  0000 C CNN
 	1    2400 1150
@@
 F 0 "C3" H 2675 1250 50  0000 L CNN
 F 1 "10n" H 2675 1050 50  0000 L CNN
-F 2 "C_0805" H 2688 1000 50  0000 C CNN
+F 2 "C_0603" H 2688 1000 50  0000 C CNN
 F 3 "" H 2650 1150 50  0000 C CNN
 	1    2650 1150
@@
 $EndComp
 $Comp
-L GND #PWR05
+L GND #PWR2
 U 1 1 58DD4181
 P 2400 1300
-F 0 "#PWR05" H 2400 1050 50  0001 C CNN
+F 0 "#PWR2" H 2400 1050 50  0001 C CNN
 F 1 "GND" H 2400 1150 50  0000 C CNN
 F 2 "" H 2400 1300 50  0000 C CNN
@@
 $EndComp
 $Comp
-L GND #PWR06
+L GND #PWR4
 U 1 1 58DD41A1
 P 2650 1300
-F 0 "#PWR06" H 2650 1050 50  0001 C CNN
+F 0 "#PWR4" H 2650 1050 50  0001 C CNN
 F 1 "GND" H 2650 1150 50  0000 C CNN
 F 2 "" H 2650 1300 50  0000 C CNN
@@
 $EndComp
 $Comp
-L +3.3V #PWR07
+L +3.3V #PWR1
 U 1 1 58DD41C1
 P 2400 1000
-F 0 "#PWR07" H 2400 850 50  0001 C CNN
+F 0 "#PWR1" H 2400 850 50  0001 C CNN
 F 1 "+3.3V" H 2400 1140 50  0000 C CNN
 F 2 "" H 2400 1000 50  0000 C CNN
@@
 $EndComp
 $Comp
-L +3.3V #PWR08
+L +3.3V #PWR3
 U 1 1 58DD41E1
 P 2650 1000
-F 0 "#PWR08" H 2650 850 50  0001 C CNN
+F 0 "#PWR3" H 2650 850 50  0001 C CNN
 F 1 "+3.3V" H 2650 1140 50  0000 C CNN
 F 2 "" H 2650 1000 50  0000 C CNN
@@
 $EndComp
 $Comp
-L CONN_01X04 P1
-U 1 1 58DD428A
-P 2900 2450
-F 0 "P1" H 2900 2700 50  0000 C CNN
-F 1 "CONN_01X04" V 3000 2450 50  0000 C CNN
-F 2 "TerminalBlock_Pheonix_MPT-2.54mm_4pol" H 2900 2450 50  0001 C CNN
-F 3 "" H 2900 2450 50  0000 C CNN
-	1    2900 2450
-	-1   0    0    -1
-$EndComp
-$Comp
-L GND #PWR09
+L GND #PWR5
 U 1 1 58DD42F2
 P 3200 2700
-F 0 "#PWR09" H 3200 2450 50  0001 C CNN
+F 0 "#PWR5" H 3200 2450 50  0001 C CNN
 F 1 "GND" H 3200 2550 50  0000 C CNN
 F 2 "" H 3200 2700 50  0000 C CNN
@@
 P 6500 1950
 F 0 "P2" H 6500 2200 50  0000 C CNN
-F 1 "CONN_01X04" V 6600 1950 50  0000 C CNN
+F 1 "SYS" V 6600 1950 50  0000 C CNN
 F 2 "TerminalBlock_Pheonix_MPT-2.54mm_4pol" H 6450 1050 50  0001 C CNN
 F 3 "" H 6500 1950 50  0000 C CNN
@@
 $EndComp
 $Comp
-L GND #PWR010
+L GND #PWR14
 U 1 1 58DD52DA
 P 6300 2000
-F 0 "#PWR010" H 6300 1750 50  0001 C CNN
+F 0 "#PWR14" H 6300 1750 50  0001 C CNN
 F 1 "GND" H 6300 1850 50  0000 C CNN
 F 2 "" H 6300 2000 50  0000 C CNN
@@
 $EndComp
 $Comp
-L +3.3V #PWR011
+L +3.3V #PWR13
 U 1 1 58DD5312
 P 6300 1800
-F 0 "#PWR011" H 6300 1650 50  0001 C CNN
+F 0 "#PWR13" H 6300 1650 50  0001 C CNN
 F 1 "+3.3V" H 6300 1940 50  0000 C CNN
 F 2 "" H 6300 1800 50  0000 C CNN
@@
 $EndComp
 $Comp
-L GND #PWR012
+L GND #PWR15
 U 1 1 58DD5379
 P 6300 2100
-F 0 "#PWR012" H 6300 1850 50  0001 C CNN
+F 0 "#PWR15" H 6300 1850 50  0001 C CNN
 F 1 "GND" H 6300 1950 50  0000 C CNN
 F 2 "" H 6300 2100 50  0000 C CNN
@@
 VG1
 $Comp
-L C C5
+L C C1
 U 1 1 58DE727D
 P 5450 1850
-F 0 "C5" H 5475 1950 50  0000 L CNN
-F 1 "18pF" H 5475 1750 50  0000 L CNN
-F 2 "C_0805" H 5488 1700 50  0001 C CNN
+F 0 "C1" H 5475 1950 50  0000 L CNN
+F 1 "36pF" H 5475 1750 50  0000 L CNN
+F 2 "C_0603" H 5488 1700 50  0001 C CNN
 F 3 "" H 5450 1850 50  0000 C CNN
 	1    5450 1850
@@
 F 0 "R4" V 5680 2400 50  0000 C CNN
 F 1 "47k" V 5600 2400 50  0000 C CNN
-F 2 "C_0805" V 5530 2400 50  0001 C CNN
+F 2 "C_0603" V 5530 2400 50  0001 C CNN
 F 3 "" H 5600 2400 50  0000 C CNN
 	1    5600 2400
@@
 F 0 "R5" V 6030 2100 50  0000 C CNN
 F 1 "4.7k" V 5950 2100 50  0000 C CNN
-F 2 "C_0805" V 5880 2100 50  0000 C CNN
+F 2 "C_0603" V 5880 2100 50  0000 C CNN
 F 3 "" H 5950 2100 50  0000 C CNN
 	1    5950 2100
@@
 	3950 2750 3950 2700
 $Comp
-L GND #PWR013
+L GND #PWR6
 U 1 1 58DE8892
 P 3950 2750
-F 0 "#PWR013" H 3950 2500 50  0001 C CNN
+F 0 "#PWR6" H 3950 2500 50  0001 C CNN
 F 1 "GND" H 3950 2600 50  0000 C CNN
 F 2 "" H 3950 2750 50  0000 C CNN
@@
 $EndComp
 $Comp
-L +3.3V #PWR014
+L +3.3V #PWR11
 U 1 1 58DE93A0
 P 5550 2700
-F 0 "#PWR014" H 5550 2550 50  0001 C CNN
+F 0 "#PWR11" H 5550 2550 50  0001 C CNN
 F 1 "+3.3V" H 5550 2840 50  0000 C CNN
 F 2 "" H 5550 2700 50  0000 C CNN
@@
 $EndComp
 $Comp
-L GND #PWR015
+L GND #PWR12
 U 1 1 58DE93D8
 P 5550 2900
-F 0 "#PWR015" H 5550 2650 50  0001 C CNN
+F 0 "#PWR12" H 5550 2650 50  0001 C CNN
 F 1 "GND" H 5550 2750 50  0000 C CNN
 F 2 "" H 5550 2900 50  0000 C CNN
@@
 	5150 2800 5550 2800
 $Comp
-L C C7
+L C C4
 U 1 1 58DE9469
 P 5150 2950
-F 0 "C7" H 5175 3050 50  0000 L CNN
+F 0 "C4" H 5175 3050 50  0000 L CNN
 F 1 "10n" H 5175 2850 50  0000 L CNN
-F 2 "C_0805" H 5188 2800 50  0001 C CNN
+F 2 "C_0603" H 5188 2800 50  0001 C CNN
 F 3 "" H 5150 2950 50  0000 C CNN
 	1    5150 2950
@@
 Connection ~ 5250 2800
 $Comp
-L GND #PWR016
+L GND #PWR10
 U 1 1 58DE9519
 P 5150 3100
-F 0 "#PWR016" H 5150 2850 50  0001 C CNN
+F 0 "#PWR10" H 5150 2850 50  0001 C CNN
 F 1 "GND" H 5150 2950 50  0000 C CNN
 F 2 "" H 5150 3100 50  0000 C CNN
@@
 Wire Wire Line
 	5750 1900 6300 1900
+$Comp
+L CONN_01X02 J1
+U 1 1 59154B49
+P 2900 2450
+F 0 "J1" H 2900 2600 50  0000 C CNN
+F 1 "PHOTO" V 3000 2450 50  0000 C CNN
+F 2 "Pin_Header_Straight_1x02_Pitch2.54mm" H 2900 2450 50  0001 C CNN
+F 3 "" H 2900 2450 50  0001 C CNN
+	1    2900 2450
+	-1   0    0    1
+$EndComp
 $EndSCHEMATC

Commit message: update schematic
Parts:
- added R3: J, C_0603, symbol R
- U1: footprint SOIC-8_3.9x4.9mm_Pitch1.27mm -> Housings_SSOP:SSOP-8_2.95x2.8mm_Pitch0.65mm
Connections:
- wire segments 27 -> 29
Changed lines of the file:
@@
 F 0 "U1" H 4700 2450 60  0000 C CNN
 F 1 "TSV992" H 4700 1950 60  0000 C CNN
-F 2 "SOIC-8_3.9x4.9mm_Pitch1.27mm" H 4700 2250 60  0001 C CNN
+F 2 "Housings_SSOP:SSOP-8_2.95x2.8mm_Pitch0.65mm" H 4700 2250 60  0001 C CNN
 F 3 "" H 4700 2250 60  0001 C CNN
 	1    4700 2200
@@
 L +3.3V #PWR13
 U 1 1 58DD5312
-P 6300 1800
-F 0 "#PWR13" H 6300 1650 50  0001 C CNN
-F 1 "+3.3V" H 6300 1940 50  0000 C CNN
-F 2 "" H 6300 1800 50  0000 C CNN
-F 3 "" H 6300 1800 50  0000 C CNN
-	1    6300 1800
+P 5950 1450
+F 0 "#PWR13" H 5950 1300 50  0001 C CNN
+F 1 "+3.3V" H 5950 1590 50  0000 C CNN
+F 2 "" H 5950 1450 50  0000 C CNN
+F 3 "" H 5950 1450 50  0000 C CNN
+	1    5950 1450
 	0    -1   -1   0
 $EndComp
@@
 	-1   0    0    1
 $EndComp
+$Comp
+L R R3
+U 1 1 59155773
+P 6100 1450
+F 0 "R3" V 6180 1450 50  0000 C CNN
+F 1 "J" V 6100 1450 50  0000 C CNN
+F 2 "C_0603" V 6030 1450 50  0001 C CNN
+F 3 "" H 6100 1450 50  0000 C CNN
+	1    6100 1450
+	0    1    1    0
+$EndComp
+Wire Wire Line
+	6250 1450 6250 1800
+Wire Wire Line
+	6250 1800 6300 1800
 $EndSCHEMATC
